Commit message: Add rigid-body slung load model (WIP)

File: models/rotors_description/urdf/iris_slung_load_base.xacro (robot description, xacro)
@@ -1,4 +1,4 @@
 <?xml version="1.0"?>
-<robot name="iris" xmlns:xacro="http://ros.org/wiki/xacro">
+<robot name="iris_slung_load" xmlns:xacro="http://ros.org/wiki/xacro">
   <!-- Properties that can be assigned at build time as arguments.
   Is there a reason not to make all properties arguments?
@@ -179,5 +179,5 @@
   <xacro:load_macro
       load_mass="0.25"
-      load_radius="0.01"
+      load_radius="0.05"
       cable_mass="0.004"
       fake_joint_mass="1e-3"

File: models/rotors_description/urdf/slung_load.xacro (robot description, xacro)
@@ -18,4 +18,16 @@
 <robot xmlns:xacro="http://ros.org/wiki/xacro">
   <!-- Property Blocks -->
+  <!-- Rigid body (load) -->
+  <xacro:property name="rb_inertia">
+    <inertia
+    ixx="${1/12 * rb_mass * (rb_height * rb_height + rb_width * rb_width)}"
+    iyy="${1/12 * rb_mass * (rb_length * rb_length + rb_height * rb_height)}"
+    izz="${1/12 * rb_mass * (rb_length * rb_length + rb_width * rb_width)}"
+    ixy="0.0" ixz="0.0" iyz="0.0" /> <!-- [kg.m^2] [kg.m^2] [kg.m^2] [kg.m^2] [kg.m^2] [kg.m^2] -->
+  </xacro:property>
+  <!-- Cable -->
+  <xacro:property name="cable_attachment_origin">
+    <origin xyz="0.0 0.0 ${cable_length/2}" />
+  </xacro:property>
   <xacro:property name="cable_inertia">
     <inertia
@@ -23,11 +35,4 @@
     iyy="${1/12 * cable_mass * (cable_length * cable_length + cable_width * cable_width)}"
     izz="${1/12 * cable_mass * (cable_width * cable_width + cable_width * cable_width)}"
-    ixy="0.0" ixz="0.0" iyz="0.0" /> <!-- [kg.m^2] [kg.m^2] [kg.m^2] [kg.m^2] [kg.m^2] [kg.m^2] -->
-  </xacro:property>
-  <xacro:property name="load_inertia">
-    <inertia
-    ixx="${2/5 * load_mass * load_radius * load_radius}"
-    iyy="${2/5 * load_mass * load_radius * load_radius}"
-    izz="${2/5 * load_mass * load_radius * load_radius}"
     ixy="0.0" ixz="0.0" iyz="0.0" /> <!-- [kg.m^2] [kg.m^2] [kg.m^2] [kg.m^2] [kg.m^2] [kg.m^2] -->
   </xacro:property>
@@ -39,15 +44,34 @@
     ixy="0.0" ixz="0.0" iyz="0.0" /> <!-- [kg.m^2] [kg.m^2] [kg.m^2] [kg.m^2] [kg.m^2] [kg.m^2] -->
   </xacro:property>
-  <!-- Main multirotor link -->
-  <xacro:macro name="load_macro"
-    params="load_mass load_radius cable_mass fake_joint_mass cable_length cable_width cable_color load_color">
-    <link name="cable_link">
+  <!-- Quad  -->
+  <xacro:property name="quad_inertia">
+    <inertia
+    ixx="${1/12 * quad_mass * (quad_height * quad_height + quad_width * quad_width)}"
+    iyy="${1/12 * quad_mass * (quad_length * quad_length + quad_height * quad_height)}"
+    izz="${1/12 * quad_mass * (quad_length * quad_length + quad_width * quad_width)}"
+    ixy="0.0" ixz="0.0" iyz="0.0" /> <!-- [kg.m^2] [kg.m^2] [kg.m^2] [kg.m^2] [kg.m^2] [kg.m^2] -->
+  </xacro:property>
+  <!-- Macro Blocks -->
+  <!-- Cable Macro -->
+  <xacro:macro name="cable_macro"
+    params="parent child cable_number *attachment_point">
+    <xacro:spherical_joint_xy
+       parent_link="${parent}"
+       child_link="cable_link_${cable_number}">
+       <xacro:insert_block name="attachment_point" />
+    </xacro:spherical_joint_xy>
+    <xacro:spherical_joint_xy
+       parent_link="cable_link_${cable_number}"
+       child_link="${child}">
+       <origin xyz="0.0 0.0 ${cable_length}" />
+    </xacro:spherical_joint_xy>
+    <link name="cable_link_${cable_number}">
       <inertial>
+        <xacro:insert_block name="cable_attachment_origin" />
         <mass value="${cable_mass}" />  <!-- [kg] -->
-        <origin xyz="0 0 ${cable_length/2}" />
         <xacro:insert_block name="cable_inertia" />
       </inertial>
       <visual>
-        <origin xyz="0 0 ${cable_length/2}" rpy="0 0 0" />
+        <xacro:insert_block name="cable_attachment_origin" />
         <geometry>
           <box size="${cable_width} ${cable_width} ${cable_length}"/> <!-- [m] [m] [m] -->
@@ -55,20 +79,68 @@
       </visual>
       <!-- <collision>
-        <origin xyz="0 0 ${cable_length/2}" rpy="0 0 0" />
         <geometry>
-          <box size="${cable_width} ${cable_width} ${cable_length}" />
+          <box size="${cable_length} ${cable_width} ${cable_length}" />
         </geometry>
       </collision> -->
     </link>
-    <link name="load_link">
+  </xacro:macro>
+  <!-- Spherical joint emulation Macro -->
+  <xacro:macro name="spherical_joint_xy"
+    params="parent_link child_link *attachment_point">
+    <link name="fake_joint_${parent_link}_${child_link}">
+        <inertial>
+            <mass value="${fake_joint_mass}" />  <!-- [kg] -->
+            <xacro:insert_block name="fake_joint_inertia" />
+        </inertial>
+        <!-- <visual>
+          <geometry>
+            <sphere radius="${0.01}"/>
+          </geometry>
+        </visual> -->
+    </link>
+    <joint name="fake_joint_${parent_link}_${child_link}_x" type="continuous">
+      <xacro:insert_block name="attachment_point" />
+      <axis xyz="1 0 0" />
+      <parent link="${parent_link}" />
+      <child link="fake_joint_${parent_link}_${child_link}" />
+    </joint>
+    <joint name="fake_joint_${parent_link}_${child_link}_y" type="continuous">
+      <axis xyz="0 1 0" />
+      <parent link="fake_joint_${parent_link}_${child_link}" />
+      <child link="${child_link}" />
+    </joint>
+  </xacro:macro>
+  <!-- Quadrotor macro -->
+    <xacro:macro name="quad_macro"
+    params="quad_number">
+    <link name="quad_link_${quad_number}">
       <inertial>
-        <mass value="${load_mass}" />  <!-- [kg] -->
-        <origin xyz="0 0 0" />
-        <xacro:insert_block name="load_inertia" />
+        <mass value="${quad_mass}" />  <!-- [kg] -->
+        <xacro:insert_block name="quad_inertia" />
       </inertial>
       <visual>
-        <origin xyz="0 0 0" rpy="0 0 0" />
         <geometry>
-          <sphere radius="${load_radius}"/> <!-- [m] -->
+          <box size="${quad_length} ${quad_width} ${quad_height}"/> <!-- [m] [m] [m] -->
+        </geometry>
+      </visual>
+      <collision>
+        <geometry>
+          <box size="${quad_length} ${quad_width} ${quad_height}"/> <!-- [m] [m] [m] -->
+        </geometry>
+      </collision>
+    </link>
+  </xacro:macro>
+  <!-- Rigid-body (load) Macro -->
+  <xacro:macro name="rb_load_macro"
+    params="rb_mass rb_length rb_width rb_height cable_mass cable_length cable_width quad_mass quad_length quad_width quad_height fake_joint_mass">
+    <link name="rb_link">
+      <inertial>
+        <mass value="${rb_mass}" />  <!-- [kg] -->
+        <origin xyz="0 0 0" />
+        <xacro:insert_block name="rb_inertia" />
+      </inertial>
+      <visual>
+        <geometry>
+          <box size="${rb_length} ${rb_width} ${rb_height}"/> <!-- [m] [m] [m] -->
         </geometry>
       </visual>
@@ -80,45 +152,33 @@
       </collision> -->
     </link>
-    <joint name="load_cable" type="fixed">
-      <origin xyz="0 0 0" rpy="0 0 0" />
-      <parent link="load_link" />
-      <child link="cable_link" />
-    </joint>
-    <xacro:spherical_joint_xy
-       parent_link="cable_link"
-       child_link="base_link">
-    </xacro:spherical_joint_xy>
-  </xacro:macro>
-  <xacro:property name="cable_origin">
-    <origin xyz="0.0 0.0 ${cable_length}" />
-  </xacro:property>
-  <!-- Main multirotor link -->
-  <xacro:macro name="spherical_joint_xy"
-    params="parent_link child_link">
-    <link name="fake_joint_${parent_link}_${child_link}">
-        <inertial>
-            <mass value="${fake_joint_mass}" />  <!-- [kg] -->
-            <origin xyz="0 0 0" rpy="0 0 0"/>
-            <xacro:insert_block name="fake_joint_inertia" />
-        </inertial>
-        <visual>
-          <origin xyz="0 0 0" rpy="0 0 0" />
-          <geometry>
-            <sphere radius="${load_radius/5}"/> <!-- [m] -->
-          </geometry>
-        </visual>
-    </link>
-    <joint name="fake_joint_${parent_link}_${child_link}_x" type="continuous">
-      <xacro:insert_block name="cable_origin" />
-      <axis xyz="1 0 0" />
-      <parent link="${parent_link}" />
-      <child link="fake_joint_${parent_link}_${child_link}" />
-    </joint>
-    <joint name="fake_joint_${parent_link}_${child_link}_y" type="continuous">
-      <origin xyz="0 0 0" rpy="0 0 0" />
-      <axis xyz="0 1 0" />
-      <parent link="fake_joint_${parent_link}_${child_link}" />
-      <child link="${child_link}" />
-    </joint>
+    <!-- Four quadrotors -->
+    <!-- <xacro:cable_macro parent="rb_link" cable_number="0">
+      <origin xyz="${rb_length/2} ${rb_width/2} ${rb_height/2}" />
+    </xacro:cable_macro>
+    <xacro:cable_macro parent="rb_link" cable_number="1">
+      <origin xyz="${-rb_length/2} ${rb_width/2} ${rb_height/2}" />
+    </xacro:cable_macro>
+    <xacro:cable_macro parent="rb_link" cable_number="2">
+      <origin xyz="${-rb_length/2} ${-rb_width/2} ${rb_height/2}" />
+    </xacro:cable_macro>
+    <xacro:cable_macro parent="rb_link" cable_number="3">
+      <origin xyz="${rb_length/2} ${-rb_width/2} ${rb_height/2}" />
+    </xacro:cable_macro> -->
+    <!-- Three quadrotors -->
+    <xacro:quad_macro quad_number="0">
+    </xacro:quad_macro>
+    <xacro:quad_macro quad_number="1">
+    </xacro:quad_macro>
+    <xacro:quad_macro quad_number="2">
+    </xacro:quad_macro>
+    <xacro:cable_macro parent="rb_link" child="quad_link_0" cable_number="0">
+      <origin xyz="${rb_length/2} ${-rb_width/2} ${rb_height/2}" />
+    </xacro:cable_macro>
+    <xacro:cable_macro parent="rb_link" child="quad_link_1" cable_number="1">
+      <origin xyz="${rb_length/2} ${rb_width/2} ${rb_height/2}" />
+    </xacro:cable_macro>
+    <xacro:cable_macro parent="rb_link" child="quad_link_2" cable_number="2">
+      <origin xyz="${-rb_length/2} ${0} ${rb_height/2}" />
+    </xacro:cable_macro>
   </xacro:macro>
 </robot>
