Commit message: Cleanup SDF models. Point mass and rigid body load from 1 to 4 vehicles.

File: models/rotors_description/urdf/point_mass_load_1_vehicle_base.xacro (robot description, xacro)
@@ -1,8 +1,8 @@
 <?xml version="1.0"?>
-<robot name="rigid_body_load_3_vehicles" xmlns:xacro="http://ros.org/wiki/xacro">
+<robot name="point_mass_load_1_vehicle" xmlns:xacro="http://ros.org/wiki/xacro">
   <!-- Properties that can be assigned at build time as arguments.
   Is there a reason not to make all properties arguments?
   -->
-  <xacro:arg name='name' default='rigid_body_load_3_vehicles' />
+  <xacro:arg name='name' default='point_mass_load_1_vehicle' />
   <xacro:arg name='mavlink_addr' default='INADDR_ANY' />
   <xacro:arg name='serial_enabled' default='false' />
@@ -26,8 +26,8 @@
   <xacro:arg name='log_file' default='iris' />
   <!-- Rigid body load -->
-  <xacro:arg name='rb_mass' default='0.75' />
-  <xacro:arg name='rb_length' default='1.2' />
-  <xacro:arg name='rb_width' default='0.8' />
-  <xacro:arg name='rb_height' default='0.2' />
+  <xacro:arg name='rb_mass' default='0.3' />
+  <xacro:arg name='rb_length' default='0.1' />
+  <xacro:arg name='rb_width' default='0.1' />
+  <xacro:arg name='rb_height' default='0.1' />
   <xacro:arg name='rb_color' default='Gold' />
   <xacro:arg name='fake_joint_mass' default='1e-3' />
@@ -39,5 +39,5 @@
   <xacro:arg name='cable_radius' default='0.01' />
   <xacro:arg name='cable_color' default='White' />
-  <!-- IRIS 0 -->
+  <!-- IRIS -->
   <xacro:property name='ID' value='0' />
   <xacro:property name="namespace" value="iris_${ID}" />
@@ -54,34 +54,5 @@
   <!-- Instantiate other iris elements -->
   <xacro:include filename="$(arg rotors_description_dir)/urdf/generic_iris_others.xacro" />
-  <!-- IRIS 1 -->
-  <xacro:property name='ID' value='1' />
-  <xacro:property name="namespace" value="iris_${ID}" />
-  <xacro:property name='base_link' value='base_link_${ID}' />
-  <xacro:property name='base_joint' value='base_joint_${ID}' />
-  <xacro:property name='mavlink_udp_port' value='1456${ID}' />
-  <xacro:property name='mavlink_tcp_port' value='456${ID}' />
-  <xacro:property name='qgc_udp_port' value='1455${ID}' />
-  <xacro:property name='sdk_udp_port' value='1454${ID}' />
-  <!-- macros for gazebo plugins, sensors -->
-  <xacro:include filename="$(arg rotors_description_dir)/urdf/generic_iris_component_snippets.xacro" />
-  <!-- Instantiate iris "mechanics" -->
-  <xacro:include filename="$(arg rotors_description_dir)/urdf/generic_iris.xacro" />
-  <!-- Instantiate other iris elements -->
-  <xacro:include filename="$(arg rotors_description_dir)/urdf/generic_iris_others.xacro" />
-  <!-- IRIS 2 -->
-  <xacro:property name='ID' value='2' />
-  <xacro:property name="namespace" value="iris_${ID}" />
-  <xacro:property name='base_link' value='base_link_${ID}' />
-  <xacro:property name='base_joint' value='base_joint_${ID}' />
-  <xacro:property name='mavlink_udp_port' value='1456${ID}' />
-  <xacro:property name='mavlink_tcp_port' value='456${ID}' />
-  <xacro:property name='qgc_udp_port' value='1455${ID}' />
-  <xacro:property name='sdk_udp_port' value='1454${ID}' />
-  <!-- macros for gazebo plugins, sensors -->
-  <xacro:include filename="$(arg rotors_description_dir)/urdf/generic_iris_component_snippets.xacro" />
-  <!-- Instantiate iris "mechanics" -->
-  <xacro:include filename="$(arg rotors_description_dir)/urdf/generic_iris.xacro" />
-  <!-- Instantiate other iris elements -->
-  <xacro:include filename="$(arg rotors_description_dir)/urdf/generic_iris_others.xacro" />
+  <!-- Rigid body and cables -->
   <xacro:include filename="$(arg rotors_description_dir)/urdf/rigid_body_load.xacro" />
   <xacro:rb_load
@@ -101,27 +72,63 @@
     fake_joint_damping="$(arg fake_joint_damping)"
     fake_joint_friction="$(arg fake_joint_friction)">
-    <origin xyz="${$(arg rb_length)/2} ${$(arg rb_width)/2} ${$(arg rb_height)/2}" />
+    <origin xyz="0.0 0.0 ${$(arg rb_height)/2}" />
   </xacro:cable_macro>
-  <xacro:cable_macro parent="rb_link" child="base_link_1" cable_number="1"
-    cable_mass="$(arg cable_mass)"
-    cable_length="$(arg cable_length)"
-    cable_radius="$(arg cable_radius)"
-    cable_color="$(arg cable_color)"
-    fake_joint_mass="$(arg fake_joint_mass)"
-    fake_joint_inertia="$(arg fake_joint_inertia)"
-    fake_joint_damping="$(arg fake_joint_damping)"
-    fake_joint_friction="$(arg fake_joint_friction)">
-    <origin xyz="${$(arg rb_length)/2} ${-$(arg rb_width)/2} ${$(arg rb_height)/2}" />
-  </xacro:cable_macro>
-  <xacro:cable_macro parent="rb_link" child="base_link_2" cable_number="2"
-    cable_mass="$(arg cable_mass)"
-    cable_length="$(arg cable_length)"
-    cable_radius="$(arg cable_radius)"
-    cable_color="$(arg cable_color)"
-    fake_joint_mass="$(arg fake_joint_mass)"
-    fake_joint_inertia="$(arg fake_joint_inertia)"
-    fake_joint_damping="$(arg fake_joint_damping)"
-    fake_joint_friction="$(arg fake_joint_friction)">
-    <origin xyz="${-$(arg rb_length)/2} ${0} ${$(arg rb_height)/2}" />
-  </xacro:cable_macro>
+  <gazebo>
+    <!-- Groundtruth plugin -->
+    <plugin name="rb_link_groundtruth" filename="libgazebo_ros_p3d.so">
+      <alwaysOn>true</alwaysOn>
+      <updateRate>50.0</updateRate>
+      <bodyName>rb_link</bodyName>
+      <topicName>odom</topicName>
+      <robotNamespace>/rb_link/</robotNamespace>
+      <!-- <gaussianNoise>0.0</gaussianNoise>
+      <frameName>map</frameName>
+      <xyzOffsets>0 0 0</xyzOffsets>
+      <rpyOffsets>0 0 0</rpyOffsets> -->
+    </plugin>
+    <plugin name="quadrotor_groundtruth" filename="libgazebo_ros_p3d.so">
+      <alwaysOn>true</alwaysOn>
+      <updateRate>50.0</updateRate>
+      <bodyName>base_link_0</bodyName>
+      <topicName>odom</topicName>
+      <robotNamespace>/quad</robotNamespace>
+      <!-- <gaussianNoise>0.0</gaussianNoise>
+      <frameName>map</frameName>
+      <xyzOffsets>0 0 0</xyzOffsets>
+      <rpyOffsets>0 0 0</rpyOffsets> -->
+    </plugin>
+    <plugin name="cable_groundtruth" filename="libgazebo_ros_p3d.so">
+      <alwaysOn>true</alwaysOn>
+      <updateRate>50.0</updateRate>
+      <bodyName>cable_link_0</bodyName>
+      <topicName>odom</topicName>
+      <robotNamespace>/cable/</robotNamespace>
+      <!-- <gaussianNoise>0.0</gaussianNoise>
+      <frameName>map</frameName>
+      <xyzOffsets>0 0 0</xyzOffsets>
+      <rpyOffsets>0 0 0</rpyOffsets> -->
+    </plugin>
+    <!-- Force plugin -->
+    <plugin name="rb_link_force" filename="libgazebo_ros_f3d.so">
+      <alwaysOn>true</alwaysOn>
+      <updateRate>50.0</updateRate>
+      <bodyName>rb_link</bodyName>
+      <topicName>force</topicName>
+      <robotNamespace>/rb_link/</robotNamespace>
+    </plugin>
+    <plugin name="quadrotor_force" filename="libgazebo_ros_f3d.so">
+      <alwaysOn>true</alwaysOn>
+      <updateRate>50.0</updateRate>
+      <bodyName>base_link_0</bodyName>
+      <topicName>force</topicName>
+      <robotNamespace>/quad/</robotNamespace>
+    </plugin>
+    <plugin name="cable_force" filename="libgazebo_ros_f3d.so">
+      <alwaysOn>true</alwaysOn>
+      <updateRate>50.0</updateRate>
+      <bodyName>cable_link_0</bodyName>
+      <topicName>force</topicName>
+      <robotNamespace>/cable/</robotNamespace>
+    </plugin>
+  </gazebo>
 </robot>

File: models/rotors_description/urdf/point_mass_load_2_vehicles_base.xacro (robot description, xacro)
@@ -1,8 +1,8 @@
 <?xml version="1.0"?>
-<robot name="rigid_body_load_4_vehicles" xmlns:xacro="http://ros.org/wiki/xacro">
+<robot name="point_mass_load_2_vehicles" xmlns:xacro="http://ros.org/wiki/xacro">
   <!-- Properties that can be assigned at build time as arguments.
   Is there a reason not to make all properties arguments?
   -->
-  <xacro:arg name='name' default='rigid_body_load_4_vehicles' />
+  <xacro:arg name='name' default='point_mass_load_2_vehicles' />
   <xacro:arg name='mavlink_addr' default='INADDR_ANY' />
   <xacro:arg name='serial_enabled' default='false' />
@@ -26,8 +26,8 @@
   <xacro:arg name='log_file' default='iris' />
   <!-- Rigid body load -->
-  <xacro:arg name='rb_mass' default='1.0' />
-  <xacro:arg name='rb_length' default='1.2' />
-  <xacro:arg name='rb_width' default='0.8' />
-  <xacro:arg name='rb_height' default='0.2' />
+  <xacro:arg name='rb_mass' default='0.5' />
+  <xacro:arg name='rb_length' default='0.1' />
+  <xacro:arg name='rb_width' default='0.1' />
+  <xacro:arg name='rb_height' default='0.1' />
   <xacro:arg name='rb_color' default='Gold' />
   <xacro:arg name='fake_joint_mass' default='1e-3' />
@@ -69,34 +69,4 @@
   <!-- Instantiate other iris elements -->
   <xacro:include filename="$(arg rotors_description_dir)/urdf/generic_iris_others.xacro" />
-  <!-- IRIS 2 -->
-  <xacro:property name='ID' value='2' />
-  <xacro:property name="namespace" value="iris_${ID}" />
-  <xacro:property name='base_link' value='base_link_${ID}' />
-  <xacro:property name='base_joint' value='base_joint_${ID}' />
-  <xacro:property name='mavlink_udp_port' value='1456${ID}' />
-  <xacro:property name='mavlink_tcp_port' value='456${ID}' />
-  <xacro:property name='qgc_udp_port' value='1455${ID}' />
-  <xacro:property name='sdk_udp_port' value='1454${ID}' />
-  <!-- macros for gazebo plugins, sensors -->
-  <xacro:include filename="$(arg rotors_description_dir)/urdf/generic_iris_component_snippets.xacro" />
-  <!-- Instantiate iris "mechanics" -->
-  <xacro:include filename="$(arg rotors_description_dir)/urdf/generic_iris.xacro" />
-  <!-- Instantiate other iris elements -->
-  <xacro:include filename="$(arg rotors_description_dir)/urdf/generic_iris_others.xacro" />
-  <!-- IRIS 3 -->
-  <xacro:property name='ID' value='3' />
-  <xacro:property name="namespace" value="iris_${ID}" />
-  <xacro:property name='base_link' value='base_link_${ID}' />
-  <xacro:property name='base_joint' value='base_joint_${ID}' />
-  <xacro:property name='mavlink_udp_port' value='1456${ID}' />
-  <xacro:property name='mavlink_tcp_port' value='456${ID}' />
-  <xacro:property name='qgc_udp_port' value='1455${ID}' />
-  <xacro:property name='sdk_udp_port' value='1454${ID}' />
-  <!-- macros for gazebo plugins, sensors -->
-  <xacro:include filename="$(arg rotors_description_dir)/urdf/generic_iris_component_snippets.xacro" />
-  <!-- Instantiate iris "mechanics" -->
-  <xacro:include filename="$(arg rotors_description_dir)/urdf/generic_iris.xacro" />
-  <!-- Instantiate other iris elements -->
-  <xacro:include filename="$(arg rotors_description_dir)/urdf/generic_iris_others.xacro" />
   <!-- Rigid body and cables -->
   <xacro:include filename="$(arg rotors_description_dir)/urdf/rigid_body_load.xacro" />
@@ -117,5 +87,5 @@
     fake_joint_damping="$(arg fake_joint_damping)"
     fake_joint_friction="$(arg fake_joint_friction)">
-    <origin xyz="${$(arg rb_length)/2} ${-$(arg rb_width)/2} ${$(arg rb_height)/2}" />
+    <origin xyz="0.0 0.0 ${$(arg rb_height)/2}" />
   </xacro:cable_macro>
   <xacro:cable_macro parent="rb_link" child="base_link_1" cable_number="1"
@@ -128,27 +98,5 @@
     fake_joint_damping="$(arg fake_joint_damping)"
     fake_joint_friction="$(arg fake_joint_friction)">
-    <origin xyz="${-$(arg rb_length)/2} ${-$(arg rb_width)/2} ${$(arg rb_height)/2}" />
-  </xacro:cable_macro>
-  <xacro:cable_macro parent="rb_link" child="base_link_2" cable_number="2"
-    cable_mass="$(arg cable_mass)"
-    cable_length="$(arg cable_length)"
-    cable_radius="$(arg cable_radius)"
-    cable_color="$(arg cable_color)"
-    fake_joint_mass="$(arg fake_joint_mass)"
-    fake_joint_inertia="$(arg fake_joint_inertia)"
-    fake_joint_damping="$(arg fake_joint_damping)"
-    fake_joint_friction="$(arg fake_joint_friction)">
-    <origin xyz="${-$(arg rb_length)/2} ${$(arg rb_width)/2} ${$(arg rb_height)/2}" />
-  </xacro:cable_macro>
-  <xacro:cable_macro parent="rb_link" child="base_link_3" cable_number="3"
-    cable_mass="$(arg cable_mass)"
-    cable_length="$(arg cable_length)"
-    cable_radius="$(arg cable_radius)"
-    cable_color="$(arg cable_color)"
-    fake_joint_mass="$(arg fake_joint_mass)"
-    fake_joint_inertia="$(arg fake_joint_inertia)"
-    fake_joint_damping="$(arg fake_joint_damping)"
-    fake_joint_friction="$(arg fake_joint_friction)">
-    <origin xyz="${$(arg rb_length)/2} ${$(arg rb_width)/2} ${$(arg rb_height)/2}" />
+    <origin xyz="0.0 0.0 ${$(arg rb_height)/2}" />
   </xacro:cable_macro>
 </robot>

File: models/rotors_description/urdf/point_mass_load_3_vehicles_base.xacro (robot description, xacro)
@@ -1,8 +1,8 @@
 <?xml version="1.0"?>
-<robot name="rigid_body_load_1_vehicle" xmlns:xacro="http://ros.org/wiki/xacro">
+<robot name="point_mass_load_3_vehicles" xmlns:xacro="http://ros.org/wiki/xacro">
   <!-- Properties that can be assigned at build time as arguments.
   Is there a reason not to make all properties arguments?
   -->
-  <xacro:arg name='name' default='rigid_body_load_1_vehicle' />
+  <xacro:arg name='name' default='point_mass_load_3_vehicles' />
   <xacro:arg name='mavlink_addr' default='INADDR_ANY' />
   <xacro:arg name='serial_enabled' default='false' />
@@ -26,5 +26,5 @@
   <xacro:arg name='log_file' default='iris' />
   <!-- Rigid body load -->
-  <xacro:arg name='rb_mass' default='0.3' />
+  <xacro:arg name='rb_mass' default='0.75' />
   <xacro:arg name='rb_length' default='0.1' />
   <xacro:arg name='rb_width' default='0.1' />
@@ -36,8 +36,8 @@
   <xacro:arg name='fake_joint_friction' default='1e-3' />
   <xacro:arg name='cable_mass' default='1e-3' />
-  <xacro:arg name='cable_length' default='0.8' />
+  <xacro:arg name='cable_length' default='1.23' />
   <xacro:arg name='cable_radius' default='0.01' />
   <xacro:arg name='cable_color' default='White' />
-  <!-- IRIS -->
+  <!-- IRIS 0 -->
   <xacro:property name='ID' value='0' />
   <xacro:property name="namespace" value="iris_${ID}" />
@@ -54,5 +54,40 @@
   <!-- Instantiate other iris elements -->
   <xacro:include filename="$(arg rotors_description_dir)/urdf/generic_iris_others.xacro" />
-  <!-- Rigid body and cables -->
+  <!-- IRIS 1 -->
+  <xacro:property name='ID' value='1' />
+  <xacro:property name="namespace" value="iris_${ID}" />
+  <xacro:property name='base_link' value='base_link_${ID}' />
+  <xacro:property name='base_joint' value='base_joint_${ID}' />
+  <xacro:property name='mavlink_udp_port' value='1456${ID}' />
+  <xacro:property name='mavlink_tcp_port' value='456${ID}' />
+  <xacro:property name='qgc_udp_port' value='1455${ID}' />
+  <xacro:property name='sdk_udp_port' value='1454${ID}' />
+  <!-- macros for gazebo plugins, sensors -->
+  <xacro:include filename="$(arg rotors_description_dir)/urdf/generic_iris_component_snippets.xacro" />
+  <!-- Instantiate iris "mechanics" -->
+  <xacro:include filename="$(arg rotors_description_dir)/urdf/generic_iris.xacro" />
+  <!-- Instantiate other iris elements -->
+  <xacro:include filename="$(arg rotors_description_dir)/urdf/generic_iris_others.xacro" />
+  <!-- IRIS 2 -->
+  <xacro:property name='ID' value='2' />
+  <xacro:property name="namespace" value="iris_${ID}" />
+  <xacro:property name='base_link' value='base_link_${ID}' />
+  <xacro:property name='base_joint' value='base_joint_${ID}' />
+  <xacro:property name='mavlink_udp_port' value='1456${ID}' />
+  <xacro:property name='mavlink_tcp_port' value='456${ID}' />
+  <xacro:property name='qgc_udp_port' value='1455${ID}' />
+  <xacro:property name='sdk_udp_port' value='1454${ID}' />
+  <!-- macros for gazebo plugins, sensors -->
+  <xacro:include filename="$(arg rotors_description_dir)/urdf/generic_iris_component_snippets.xacro" />
+  <!-- Instantiate iris "mechanics" -->
+  <xacro:include filename="$(arg rotors_description_dir)/urdf/generic_iris.xacro" />
+  <!-- Instantiate other iris elements -->
+  <xacro:include filename="$(arg rotors_description_dir)/urdf/generic_iris_others.xacro" />
+  <!-- Fake joints so urdf2sdf does not collapse the baselinks -->
+  <!-- <joint name="inter_base_joint_1" type="floating">
+    <origin xyz="1 1 0" />
+    <parent link="base_link_0" />
+    <child link="base_link_1" />
+  </joint> -->
   <xacro:include filename="$(arg rotors_description_dir)/urdf/rigid_body_load.xacro" />
   <xacro:rb_load
@@ -74,61 +109,25 @@
     <origin xyz="0.0 0.0 ${$(arg rb_height)/2}" />
   </xacro:cable_macro>
-  <gazebo>
-    <!-- Groundtruth plugin -->
-    <plugin name="rb_link_groundtruth" filename="libgazebo_ros_p3d.so">
-      <alwaysOn>true</alwaysOn>
-      <updateRate>50.0</updateRate>
-      <bodyName>rb_link</bodyName>
-      <topicName>odom</topicName>
-      <robotNamespace>/rb_link/</robotNamespace>
-      <!-- <gaussianNoise>0.0</gaussianNoise>
-      <frameName>map</frameName>
-      <xyzOffsets>0 0 0</xyzOffsets>
-      <rpyOffsets>0 0 0</rpyOffsets> -->
-    </plugin>
-    <plugin name="quadrotor_groundtruth" filename="libgazebo_ros_p3d.so">
-      <alwaysOn>true</alwaysOn>
-      <updateRate>50.0</updateRate>
-      <bodyName>base_link_0</bodyName>
-      <topicName>odom</topicName>
-      <robotNamespace>/quad</robotNamespace>
-      <!-- <gaussianNoise>0.0</gaussianNoise>
-      <frameName>map</frameName>
-      <xyzOffsets>0 0 0</xyzOffsets>
-      <rpyOffsets>0 0 0</rpyOffsets> -->
-    </plugin>
-    <plugin name="cable_groundtruth" filename="libgazebo_ros_p3d.so">
-      <alwaysOn>true</alwaysOn>
-      <updateRate>50.0</updateRate>
-      <bodyName>cable_link_0</bodyName>
-      <topicName>odom</topicName>
-      <robotNamespace>/cable/</robotNamespace>
-      <gaussianNoise>0.0</gaussianNoise>
-      <frameName>map</frameName>
-      <xyzOffsets>0 0 0</xyzOffsets>
-      <rpyOffsets>0 0 0</rpyOffsets>
-    </plugin>
-    <!-- Force plugin -->
-    <plugin name="rb_link_force" filename="libgazebo_ros_f3d.so">
-      <alwaysOn>true</alwaysOn>
-      <updateRate>50.0</updateRate>
-      <bodyName>rb_link</bodyName>
-      <topicName>force</topicName>
-      <robotNamespace>/rb_link/</robotNamespace>
-    </plugin>
-    <plugin name="quadrotor_force" filename="libgazebo_ros_f3d.so">
-      <alwaysOn>true</alwaysOn>
-      <updateRate>50.0</updateRate>
-      <bodyName>base_link_0</bodyName>
-      <topicName>force</topicName>
-      <robotNamespace>/quad/</robotNamespace>
-    </plugin>
-    <plugin name="cable_force" filename="libgazebo_ros_f3d.so">
-      <alwaysOn>true</alwaysOn>
-      <updateRate>50.0</updateRate>
-      <bodyName>cable_link_0</bodyName>
-      <topicName>force</topicName>
-      <robotNamespace>/cable/</robotNamespace>
-    </plugin>
-  </gazebo>
+  <xacro:cable_macro parent="rb_link" child="base_link_1" cable_number="1"
+    cable_mass="$(arg cable_mass)"
+    cable_length="$(arg cable_length)"
+    cable_radius="$(arg cable_radius)"
+    cable_color="$(arg cable_color)"
+    fake_joint_mass="$(arg fake_joint_mass)"
+    fake_joint_inertia="$(arg fake_joint_inertia)"
+    fake_joint_damping="$(arg fake_joint_damping)"
+    fake_joint_friction="$(arg fake_joint_friction)">
+    <origin xyz="0.0 0.0 ${$(arg rb_height)/2}" />
+  </xacro:cable_macro>
+  <xacro:cable_macro parent="rb_link" child="base_link_2" cable_number="2"
+    cable_mass="$(arg cable_mass)"
+    cable_length="$(arg cable_length)"
+    cable_radius="$(arg cable_radius)"
+    cable_color="$(arg cable_color)"
+    fake_joint_mass="$(arg fake_joint_mass)"
+    fake_joint_inertia="$(arg fake_joint_inertia)"
+    fake_joint_damping="$(arg fake_joint_damping)"
+    fake_joint_friction="$(arg fake_joint_friction)">
+    <origin xyz="0.0 0.0 ${$(arg rb_height)/2}" />
+  </xacro:cable_macro>
 </robot>

File: models/rotors_description/urdf/point_mass_load_4_vehicles_base.xacro (robot description, xacro)
@@ -1,8 +1,8 @@
 <?xml version="1.0"?>
-<robot name="rigid_body_load_4_vehicles" xmlns:xacro="http://ros.org/wiki/xacro">
+<robot name="point_mass_load_4_vehicles" xmlns:xacro="http://ros.org/wiki/xacro">
   <!-- Properties that can be assigned at build time as arguments.
   Is there a reason not to make all properties arguments?
   -->
-  <xacro:arg name='name' default='rigid_body_load_4_vehicles' />
+  <xacro:arg name='name' default='point_mass_load_4_vehicles' />
   <xacro:arg name='mavlink_addr' default='INADDR_ANY' />
   <xacro:arg name='serial_enabled' default='false' />
@@ -27,7 +27,7 @@
   <!-- Rigid body load -->
   <xacro:arg name='rb_mass' default='1.0' />
-  <xacro:arg name='rb_length' default='1.2' />
-  <xacro:arg name='rb_width' default='0.8' />
-  <xacro:arg name='rb_height' default='0.2' />
+  <xacro:arg name='rb_length' default='0.1' />
+  <xacro:arg name='rb_width' default='0.1' />
+  <xacro:arg name='rb_height' default='0.1' />
   <xacro:arg name='rb_color' default='Gold' />
   <xacro:arg name='fake_joint_mass' default='1e-3' />
@@ -117,5 +117,5 @@
     fake_joint_damping="$(arg fake_joint_damping)"
     fake_joint_friction="$(arg fake_joint_friction)">
-    <origin xyz="${$(arg rb_length)/2} ${-$(arg rb_width)/2} ${$(arg rb_height)/2}" />
+    <origin xyz="0.0 0.0 ${$(arg rb_height)/2}" />
   </xacro:cable_macro>
   <xacro:cable_macro parent="rb_link" child="base_link_1" cable_number="1"
@@ -128,5 +128,5 @@
     fake_joint_damping="$(arg fake_joint_damping)"
     fake_joint_friction="$(arg fake_joint_friction)">
-    <origin xyz="${-$(arg rb_length)/2} ${-$(arg rb_width)/2} ${$(arg rb_height)/2}" />
+    <origin xyz="0.0 0.0 ${$(arg rb_height)/2}" />
   </xacro:cable_macro>
   <xacro:cable_macro parent="rb_link" child="base_link_2" cable_number="2"
@@ -139,5 +139,5 @@
     fake_joint_damping="$(arg fake_joint_damping)"
     fake_joint_friction="$(arg fake_joint_friction)">
-    <origin xyz="${-$(arg rb_length)/2} ${$(arg rb_width)/2} ${$(arg rb_height)/2}" />
+    <origin xyz="0.0 0.0 ${$(arg rb_height)/2}" />
   </xacro:cable_macro>
   <xacro:cable_macro parent="rb_link" child="base_link_3" cable_number="3"
@@ -150,5 +150,5 @@
     fake_joint_damping="$(arg fake_joint_damping)"
     fake_joint_friction="$(arg fake_joint_friction)">
-    <origin xyz="${$(arg rb_length)/2} ${$(arg rb_width)/2} ${$(arg rb_height)/2}" />
+    <origin xyz="0.0 0.0 ${$(arg rb_height)/2}" />
   </xacro:cable_macro>
 </robot>
