Commit message: Remove wind and setup a (non-crashing) accurate simulation

File: models/rotors_description/urdf/rigid_body_load.xacro (robot description, xacro)
@@ -1,4 +1,6 @@
 <?xml version="1.0"?>
 <robot xmlns:xacro="http://ros.org/wiki/xacro">
+  <xacro:property name='fake_joint_damping' value='0.0' />
+  <xacro:property name='fake_joint_friction' value='0.0' />
   <!-- Rigid body load -->
   <xacro:property name="rb_inertia">
@@ -87,5 +89,5 @@
       <parent link="${parent_link}" />
       <child link="fake_joint_${parent_link}_${child_link}" />
-      <dynamics damping="0.001" friction="0.001"/>
+      <dynamics damping="${fake_joint_damping}" friction="${fake_joint_friction}"/>
     </joint>
     <joint name="fake_joint_${parent_link}_${child_link}_y" type="continuous">
@@ -93,5 +95,5 @@
       <parent link="fake_joint_${parent_link}_${child_link}" />
       <child link="${child_link}" />
-      <dynamics damping="0.001" friction="0.001"/>
+      <dynamics damping="${fake_joint_damping}" friction="${fake_joint_friction}"/>
     </joint>
   </xacro:macro>
@@ -114,5 +116,5 @@
       <parent link="${parent_link}" />
       <child link="fake_joint_${parent_link}_${child_link}" />
-      <dynamics damping="0.001" friction="0.001"/>
+      <dynamics damping="${fake_joint_damping}" friction="${fake_joint_friction}"/>
     </joint>
     <joint name="fake_joint_${parent_link}_${child_link}_x" type="continuous">
@@ -120,5 +122,5 @@
       <parent link="fake_joint_${parent_link}_${child_link}" />
       <child link="${child_link}" />
-      <dynamics damping="0.001" friction="0.001"/>
+      <dynamics damping="${fake_joint_damping}" friction="${fake_joint_friction}"/>
     </joint>
   </xacro:macro>

Commit message: Add gazebo sensors and joint damping/friction

File: models/rotors_description/urdf/rigid_body_load.xacro (robot description, xacro)
@@ -1,6 +1,4 @@
 <?xml version="1.0"?>
 <robot xmlns:xacro="http://ros.org/wiki/xacro">
-  <xacro:property name='fake_joint_damping' value='0.0' />
-  <xacro:property name='fake_joint_friction' value='0.0' />
   <!-- Rigid body load -->
   <xacro:property name="rb_inertia">
@@ -32,5 +30,5 @@
   <!-- Cable Macro -->
   <xacro:macro name="cable_macro"
-    params="parent child cable_number cable_mass cable_length cable_radius cable_color fake_joint_mass fake_joint_inertia *attachment_point">
+    params="parent child cable_number cable_mass cable_length cable_radius cable_color fake_joint_mass fake_joint_damping fake_joint_friction fake_joint_inertia *attachment_point">
     <xacro:spherical_joint_xy
        parent_link="${parent}"
@@ -97,4 +95,14 @@
       <dynamics damping="${fake_joint_damping}" friction="${fake_joint_friction}"/>
     </joint>
+    <gazebo reference="fake_joint_${parent_link}_${child_link}_x">
+      <sensor name="force_torque" type="force_torque">
+            <update_rate>50</update_rate>
+      </sensor>
+    </gazebo>
+    <gazebo reference="fake_joint_${parent_link}_${child_link}_y">
+      <sensor name="force_torque" type="force_torque">
+            <update_rate>50</update_rate>
+      </sensor>
+    </gazebo>
   </xacro:macro>
   <xacro:macro name="spherical_joint_yx"
@@ -124,4 +132,14 @@
       <dynamics damping="${fake_joint_damping}" friction="${fake_joint_friction}"/>
     </joint>
+    <gazebo reference="fake_joint_${parent_link}_${child_link}_x">
+      <sensor name="force_torque" type="force_torque">
+            <update_rate>50</update_rate>
+      </sensor>
+    </gazebo>
+    <gazebo reference="fake_joint_${parent_link}_${child_link}_y">
+      <sensor name="force_torque" type="force_torque">
+            <update_rate>50</update_rate>
+      </sensor>
+    </gazebo>
   </xacro:macro>
   <!-- Rigid-body load Macro -->
@@ -146,4 +164,9 @@
     </link>
     <gazebo reference="rb_link">
+      <sensor name="force_torque" type="force_torque">
+            <update_rate>50</update_rate>
+      </sensor>
+    </gazebo>
+    <gazebo reference="rb_link">
       <material>Gazebo/${rb_color}</material>
     </gazebo>

File: models/rotors_description/urdf/rigid_body_load_1_vehicle_base.xacro (robot description, xacro)
@@ -33,4 +33,6 @@
   <xacro:arg name='fake_joint_mass' default='1e-3' />
   <xacro:arg name='fake_joint_inertia' default='1e-3' />
+  <xacro:arg name='fake_joint_damping' default='1e-3' />
+  <xacro:arg name='fake_joint_friction' default='1e-3' />
   <xacro:arg name='cable_mass' default='1e-3' />
   <xacro:arg name='cable_length' default='0.8' />
@@ -67,6 +69,13 @@
     cable_color="$(arg cable_color)"
     fake_joint_mass="$(arg fake_joint_mass)"
-    fake_joint_inertia="$(arg fake_joint_inertia)">
+    fake_joint_inertia="$(arg fake_joint_inertia)"
+    fake_joint_damping="$(arg fake_joint_damping)"
+    fake_joint_friction="$(arg fake_joint_friction)">
     <origin xyz="0.0 0.0 ${$(arg rb_height)/2}" />
   </xacro:cable_macro>
+    <gazebo reference="base_link_0">
+      <sensor name="force_torque" type="force_torque">
+            <update_rate>50</update_rate>
+      </sensor>
+    </gazebo>
 </robot>

Commit message: FIXME: Dirty fix for multiple quadrotors with PX4_SIM_SPEED_FACTOR != 1
See https://github.com/PX4/sitl_gazebo/issues/336

File: models/rotors_description/urdf/rigid_body_load.xacro (robot description, xacro)
@@ -57,10 +57,10 @@
         </geometry>
       </visual>
-      <collision>
+      <!-- <collision>
         <xacro:insert_block name="cable_attachment_origin" />
         <geometry>
           <cylinder length="${cable_length}" radius="${cable_radius}"/>
         </geometry>
-      </collision>
+      </collision> -->
     </link>
     <gazebo reference="cable_link_${cable_number}">
