Commit message: Make Iris vehicle faster (reduce motor first-order filter pole)

File: models/rotors_description/urdf/generic_iris.xacro (robot description, xacro)
@@ -19,11 +19,15 @@
   <xacro:property name="motor_constant" value="8.54858e-06" /> <!-- [kg.m/s^2] -->
   <xacro:property name="moment_constant" value="0.06" /> <!-- [m] -->
-  <xacro:property name="time_constant_up" value="0.0125" /> <!-- [s] -->
-  <xacro:property name="time_constant_down" value="0.025" /> <!-- [s] -->
+  <xacro:property name="time_constant_up" value="0.005" />
+  <xacro:property name="time_constant_down" value="0.01" />
+  <!-- <xacro:property name="time_constant_up" value="0.0125" />
+  <xacro:property name="time_constant_down" value="0.025" /> -->
   <xacro:property name="max_rot_velocity" value="1100" /> <!-- [rad/s] -->
   <xacro:property name="sin30" value="0.5" />
   <xacro:property name="cos30" value="0.866025403784" />
   <xacro:property name="sqrt2" value="1.4142135623730951" />
-  <xacro:property name="rotor_drag_coefficient" value="8.06428e-04" />
+  <!-- <xacro:property name="rotor_drag_coefficient" value="8.06428e-04" /> -->
+  <xacro:property name="rotor_drag_coefficient" value="8.06428e-08" />
+  <!-- <xacro:property name="rotor_drag_coefficient" value="8.06428e-10" /> -->
   <xacro:property name="rolling_moment_coefficient" value="0.000001" />
   <xacro:property name="color" value="$(arg visual_material)" />
